Commit message: add paddle to urdf

File: urdf/g1_dual_arm.urdf (robot description, URDF)
Before this commit: robot g1_dual_arm, 26 links, 25 joints
Links:
- added link left_paddle, mass 0.18; collision box size=0.28 0.02 0.16; visual mesh filename=package://g1_description/meshes/left_paddle.STL
Joints:
- added joint left_hand_to_pingpong_paddle: type fixed, parent left_rubber_hand, child left_paddle, origin xyz=0.10 0.00 0.00 rpy=0 0 1.57
